File: VSlideMPad/VSlideMPad.kicad_sch (KiCad schematic)
At the start: 13 parts, among them SW1 SW_Push, SW2 SW_Push, SW3 SW_Push, SW4 SW_Push, U1 MC14490DWG

Commit message: Small layout change
Parts:
- added TP1: +5V, symbol 4ms_Connector:TestPoint
- added TP2: GND, symbol 4ms_Connector:TestPoint
Connections:
- net +5V: now also TP1.1
- net GND: now also TP2.1
Other:
- moved on the sheet: R5, R6

Commit message: V1 FABRICATED
Parts:
- C1: value 10n -> 6.7n
- TP1, TP2: footprint (none) -> 4ms_TestPoint:TestPoint_Pad_06
Changed lines of the file:
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@@
 			)
 		)
-		(property "Footprint" ""
+		(property "Footprint" "4ms_TestPoint:TestPoint_Pad_06"
 			(at 144.78 38.1 0)
 			(effects
@@
 			)
 		)
-		(property "Value" "10n"
+		(property "Value" "6.7n"
 			(at 98.806 109.728 90)
 			(effects
@@
 			)
 		)
-		(property "Footprint" ""
+		(property "Footprint" "4ms_TestPoint:TestPoint_Pad_06"
 			(at 121.92 38.1 0)
 			(effects
